Commit message: Add files via upload

File: quadruped/resources/custom_robot.urdf (robot description, URDF)
Before this commit: robot quadruped, 15 links, 14 joints
Links:
- added link hoove1, mass 0.00001; collision sphere radius=0.001; visual sphere radius=0.005
- added link hoove2, mass 0.00001; collision sphere radius=0.001; visual sphere radius=0.005
- added link hoove3, mass 0.00001; collision sphere radius=0.001; visual sphere radius=0.005
- added link hoove4, mass 0.00001; collision sphere radius=0.001; visual sphere radius=0.005
Joints:
- added joint leg-hoove1: type fixed, parent leg1, child hoove1, origin xyz=0 -0.005 -0.105
- added joint leg-hoove2: type fixed, parent leg2, child hoove2, origin xyz=0 0.005 -0.105
- added joint leg-hoove3: type fixed, parent leg3, child hoove3, origin xyz=0 -0.005 -0.105
- added joint leg-hoove4: type fixed, parent leg4, child hoove4, origin xyz=0 0.005 -0.105
- joint flange-thigh1: limit lower=0 upper=0.5 effort=10 velocity=10 -> lower=-0.5 upper=0.5 effort=10 velocity=10; origin xyz=0 0.07 0 -> xyz=0 0.07 0 rpy=0 0.5 0
- joint flange-thigh2: limit lower=0 upper=0.5 effort=10 velocity=10 -> lower=-0.5 upper=0.5 effort=10 velocity=10; origin xyz=0 -0.07 0 -> xyz=0 -0.07 0 rpy=0 0.5 0
- joint flange-thigh3: limit lower=0 upper=0.5 effort=10 velocity=10 -> lower=-0.5 upper=0.5 effort=10 velocity=10; origin xyz=0 0.07 0 -> xyz=0 0.07 0 rpy=0 -0.5 0
- joint flange-thigh4: limit lower=0 upper=0.5 effort=10 velocity=10 -> lower=-0.5 upper=0.5 effort=10 velocity=10; origin xyz=0 -0.07 0 -> xyz=0 -0.07 0 rpy=0 -0.5 0
- joint head-flange1: limit lower=-0.5 upper=0.5 effort=10 velocity=10 -> lower=-0.2 upper=0.5 effort=10 velocity=10
- joint head-flange2: limit lower=-0.5 upper=0.5 effort=10 velocity=10 -> lower=-0.2 upper=0.5 effort=10 velocity=10
- joint spine-head: type revolute -> fixed
- joint spine-tail: type revolute -> fixed
- joint tail-flange3: limit lower=-0.5 upper=0.5 effort=10 velocity=10 -> lower=-0.2 upper=0.5 effort=10 velocity=10
- joint tail-flange4: limit lower=-0.5 upper=0.5 effort=10 velocity=10 -> lower=-0.2 upper=0.5 effort=10 velocity=10
- joint thigh-leg1: limit lower=0 upper=0.5 effort=10 velocity=10 -> lower=-0.5 upper=0.5 effort=10 velocity=10; origin xyz=0 0 -0.1 -> xyz=0 0 -0.1 rpy=0 -1 0
- joint thigh-leg2: limit lower=0 upper=0.5 effort=10 velocity=10 -> lower=-0.5 upper=0.5 effort=10 velocity=10; origin xyz=0 0 -0.1 -> xyz=0 0 -0.1 rpy=0 -1 0
- joint thigh-leg3: limit lower=0 upper=0.5 effort=10 velocity=10 -> lower=-0.5 upper=0.5 effort=10 velocity=10; origin xyz=0 0 -0.1 -> xyz=0 0 -0.1 rpy=0 1 0
- joint thigh-leg4: limit lower=0 upper=0.5 effort=10 velocity=10 -> lower=-0.5 upper=0.5 effort=10 velocity=10; origin xyz=0 0 -0.1 -> xyz=0 0 -0.1 rpy=0 1 0
